File: Design/H0AR9.sch (EAGLE design)
At the start: 31 parts, among them P1 HEXABIT_17.32, U1 STM32G0B1CEU6NUFQFPN48_STM32_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, U2 PANASONIC_EKMC1601111PANASONI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, U3 BROADCOM_APDS-9950BROADCOM_AP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, U4 TEXAS_INSTRUMENTS_HDC1080DMBT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, X1 8MH

Commit message: -Standarize the files and folders
Other:
- note added: "H0AR9"
- note added: "H0AR9_Backend"
- note added: "H0AR9_Frontend"
- note removed: "Esraa Alkadour"
- note removed: "H0AR91"
- note removed: "H0AR91_Backend"
- note removed: "H0AR91_Frontend"
